File: hardware/Display/Display.kicad_pcb (KiCad board)
At the start: 2 copper layers, 78.5 x 46.2 mm, 10 parts, among them J1 Motherboard Connector, J2 SPI 128x64 SSH1106 OLED, SW1 SW_Push, SW2 SW_Push, SW3 SW_Push, SW4 SW_Push

Commit message: Update hardware pcbs
Parts:
- added G***: LOGO, Genesynth:thea, F.Cu at (163.0, 125.5)
- added G***: LOGO, LocalDisplay:nei, F.Cu at (157.0, 106.7)
- added G***: LOGO, LocalDisplay:nei, B.Cu at (156.1, 106.8)
- renumbered J2 to Display, SW3 to Down, SW4 to Left, SW2 to Right, SW1 to Up
Other:
- board text added: "+5V"
- board text added: "BTN1"
- board text added: "BTN2"
- board text added: "BTN3"
- board text added: "BTN4"
- board text added: "CC BY SA 4.0"
- board text added: "CLK"
- board text added: "CS"
- board text added: "DC"
- board text added: "GND"
- board text added: "MOSI"
- board text added: "RES"
- board text added: "Synth Display Board"
- board text added: "thea.codes"
