File: hardware/Genesynth/Genesynth.kicad_pcb (KiCad board)
At the start: 2 copper layers, 72.6 x 64 mm, 23 parts, among them J1 Audio Daughterboard, J2 Display Daughterboard, J3 POWER_JACK, U1 Teensy3.5, U2 YM2612, U3 LD1117S50 (Digital), U4 LD1117S50 (Analog)

Commit message: Updating motherboard
Parts:
- added C5: 100nF, Capacitor_THT:C_Disc_D7.0mm_W2.5mm_P5.00mm, F.Cu at (141.2, 124.7)
- added C6: 100nF, Capacitor_THT:C_Disc_D7.0mm_W2.5mm_P5.00mm, F.Cu at (144.0, 124.7)
- moved C4 2.28 mm to (142.2, 87.9), turned to 180 degrees
Routing:
- net +5V: track 105.2 -> 109.0 mm
- net +5VA: track 64.2 -> 66.2 mm
Changed lines of the file:
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@@
     (thickness 1.6)
     (drawings 25)
-    (tracks 161)
+    (tracks 168)
     (zones 0)
-    (modules 23)
+    (modules 25)
     (nets 56)
   )
@@
     (45 Margin user)
     (46 B.CrtYd user hide)
-    (47 F.CrtYd user hide)
+    (47 F.CrtYd user)
     (48 B.Fab user hide)
     (49 F.Fab user hide)
   )
   (setup
-    (last_trace_width 0.1778)
+    (last_trace_width 0.508)
     (user_trace_width 0.508)
     (trace_clearance 0.1778)
@@
   )
   (module Capacitor_THT:CP_Radial_D6.3mm_P2.50mm (layer F.Cu)
-    (at 140.4342 86.487 270)
+    (at 142.24 87.884 180)
     (descr "CP, Radial series, Radial, pin pitch=2.50mm, , diameter=6.3mm, Electrolytic Capacitor")
     (tags "CP Radial series Radial pin pitch 2.50mm  diameter 6.3mm Electrolytic Capacitor")
-    (fp_text reference C4 (at 4.191 -3.0758) (layer F.SilkS)
+    (fp_text reference C4 (at 4.191 -3.0758 -90) (layer F.SilkS)
       (effects (font (size 1 1) (thickness 0.15)))
     )
-    (fp_text value 10uF (at 1.25 4.4 270) (layer F.Fab)
+    (fp_text value 10uF (at 1.25 4.4 180) (layer F.Fab)
       (effects (font (size 1 1) (thickness 0.15)))
     )
-    (fp_text user %R (at 1.25 0 270) (layer F.Fab)
+    (fp_text user %R (at 1.25 0 180) (layer F.Fab)
       (effects (font (size 1 1) (thickness 0.15)))
     )
@@
     (fp_circle (center 1.25 0) (end 4.52 0) (layer F.SilkS) (width 0.12))
     (fp_circle (center 1.25 0) (end 4.4 0) (layer F.Fab) (width 0.1))
-    (pad 2 thru_hole circle (at 2.5 0 270) (size 1.6 1.6) (drill 0.8) (layers *.Cu *.Mask)
+    (pad 2 thru_hole circle (at 2.5 0 180) (size 1.6 1.6) (drill 0.8) (layers *.Cu *.Mask)
       (net 40 GND))
-    (pad 1 thru_hole rect (at 0 0 270) (size 1.6 1.6) (drill 0.8) (layers *.Cu *.Mask)
+    (pad 1 thru_hole rect (at 0 0 180) (size 1.6 1.6) (drill 0.8) (layers *.Cu *.Mask)
       (net 42 +5VA))
     (model ${KISYS3DMOD}/Capacitor_THT.3dshapes/CP_Radial_D6.3mm_P2.50mm.wrl
@@
     (pad 1 np_thru_hole circle (at 0 0) (size 3.2 3.2) (drill 3.2) (layers *.Cu *.Mask))
   )
-  (gr_text v0 (at 155.484762 126.928745) (layer F.SilkS)
-    (effects (font (size 1 1) (thickness 0.25)))
+  (module Capacitor_THT:C_Disc_D7.0mm_W2.5mm_P5.00mm (layer F.Cu)
+    (at 141.224 124.714 180)
+    (descr "C, Disc series, Radial, pin pitch=5.00mm, , diameter*width=7*2.5mm^2, Capacitor, http://cdn-reichelt.de/documents/datenblatt/B300/DS_KERKO_TC.pdf")
+    (tags "C Disc series Radial pin pitch 5.00mm  diameter 7mm width 2.5mm Capacitor")
+    (fp_text reference C5 (at 2.54 0 180) (layer F.SilkS)
+      (effects (font (size 1 1) (thickness 0.15)))
+    )
+    (fp_text value 100nF (at 2.5 2.5 180) (layer F.Fab)
+      (effects (font (size 1 1) (thickness 0.15)))
+    )
+    (fp_text user %R (at 2.5 0 180) (layer F.Fab)
+      (effects (font (size 1 1) (thickness 0.15)))
+    )
+    (fp_line (start 6.25 -1.5) (end -1.25 -1.5) (layer F.CrtYd) (width 0.05))
+    (fp_line (start 6.25 1.5) (end 6.25 -1.5) (layer F.CrtYd) (width 0.05))
+    (fp_line (start -1.25 1.5) (end 6.25 1.5) (layer F.CrtYd) (width 0.05))
+    (fp_line (start -1.25 -1.5) (end -1.25 1.5) (layer F.CrtYd) (width 0.05))
+    (fp_line (start 6.12 -1.37) (end 6.12 1.37) (layer F.SilkS) (width 0.12))
+    (fp_line (start -1.12 -1.37) (end -1.12 1.37) (layer F.SilkS) (width 0.12))
+    (fp_line (start -1.12 1.37) (end 6.12 1.37) (layer F.SilkS) (width 0.12))
+    (fp_line (start -1.12 -1.37) (end 6.12 -1.37) (layer F.SilkS) (width 0.12))
+    (fp_line (start 6 -1.25) (end -1 -1.25) (layer F.Fab) (width 0.1))
+    (fp_line (start 6 1.25) (end 6 -1.25) (layer F.Fab) (width 0.1))
+    (fp_line (start -1 1.25) (end 6 1.25) (layer F.Fab) (width 0.1))
+    (fp_line (start -1 -1.25) (end -1 1.25) (layer F.Fab) (width 0.1))
+    (pad 2 thru_hole circle (at 5 0 180) (size 1.6 1.6) (drill 0.8) (layers *.Cu *.Mask)
+      (net 40 GND))
+    (pad 1 thru_hole circle (at 0 0 180) (size 1.6 1.6) (drill 0.8) (layers *.Cu *.Mask)
+      (net 41 +5V))
+    (model ${KISYS3DMOD}/Capacitor_THT.3dshapes/C_Disc_D7.0mm_W2.5mm_P5.00mm.wrl
+      (at (xyz 0 0 0))
+      (scale (xyz 1 1 1))
+      (rotate (xyz 0 0 0))
+    )
   )
-  (gr_text "CC BY SA 4.0" (at 138.43 129.032) (layer F.SilkS)
-    (effects (font (size 1 1) (thickness 0.25)))
+  (module Capacitor_THT:C_Disc_D7.0mm_W2.5mm_P5.00mm (layer F.Cu)
+    (at 144.018 124.714)
+    (descr "C, Disc series, Radial, pin pitch=5.00mm, , diameter*width=7*2.5mm^2, Capacitor, http://cdn-reichelt.de/documents/datenblatt/B300/DS_KERKO_TC.pdf")
+    (tags "C Disc series Radial pin pitch 5.00mm  diameter 7mm width 2.5mm Capacitor")
+    (fp_text reference C6 (at 2.54 0) (layer F.SilkS)
+      (effects (font (size 1 1) (thickness 0.15)))
+    )
+    (fp_text value 100nF (at 2.5 2.5) (layer F.Fab)
+      (effects (font (size 1 1) (thickness 0.15)))
+    )
+    (fp_line (start -1 -1.25) (end -1 1.25) (layer F.Fab) (width 0.1))
+    (fp_line (start -1 1.25) (end 6 1.25) (layer F.Fab) (width 0.1))
+    (fp_line (start 6 1.25) (end 6 -1.25) (layer F.Fab) (width 0.1))
+    (fp_line (start 6 -1.25) (end -1 -1.25) (layer F.Fab) (width 0.1))
+    (fp_line (start -1.12 -1.37) (end 6.12 -1.37) (layer F.SilkS) (width 0.12))
+    (fp_line (start -1.12 1.37) (end 6.12 1.37) (layer F.SilkS) (width 0.12))
+    (fp_line (start -1.12 -1.37) (end -1.12 1.37) (layer F.SilkS) (width 0.12))
+    (fp_line (start 6.12 -1.37) (end 6.12 1.37) (layer F.SilkS) (width 0.12))
+    (fp_line (start -1.25 -1.5) (end -1.25 1.5) (layer F.CrtYd) (width 0.05))
+    (fp_line (start -1.25 1.5) (end 6.25 1.5) (layer F.CrtYd) (width 0.05))
+    (fp_line (start 6.25 1.5) (end 6.25 -1.5) (layer F.CrtYd) (width 0.05))
+    (fp_line (start 6.25 -1.5) (end -1.25 -1.5) (layer F.CrtYd) (width 0.05))
+    (fp_text user %R (at 2.5 0) (layer F.Fab)
+      (effects (font (size 1 1) (thickness 0.15)))
+    )
+    (pad 1 thru_hole circle (at 0 0) (size 1.6 1.6) (drill 0.8) (layers *.Cu *.Mask)
+      (net 42 +5VA))
+    (pad 2 thru_hole circle (at 5 0) (size 1.6 1.6) (drill 0.8) (layers *.Cu *.Mask)
+      (net 40 GND))
+    (model ${KISYS3DMOD}/Capacitor_THT.3dshapes/C_Disc_D7.0mm_W2.5mm_P5.00mm.wrl
+      (at (xyz 0 0 0))
+      (scale (xyz 1 1 1))
+      (rotate (xyz 0 0 0))
+    )
+  )
+  (gr_text v0 (at 153.601072 127.254) (layer F.SilkS)
+    (effects (font (size 0.7 0.7) (thickness 0.175)))
+  )
+  (gr_text "CC BY SA 4.0" (at 145.853869 127.254) (layer F.SilkS)
+    (effects (font (size 0.7 0.7) (thickness 0.175)))
   )
-  (gr_text thea.codes (at 137.287143 126.928745) (layer F.SilkS)
-    (effects (font (size 1 1) (thickness 0.25)))
+  (gr_text thea.codes (at 135.89 127.254) (layer F.SilkS)
+    (effects (font (size 0.7 0.7) (thickness 0.175)))
   )
-  (gr_text "GeneSynth Motherboard" (at 144.802619 124.55399) (layer F.SilkS)
-    (effects (font (size 1.3 1.3) (thickness 0.3)))
+  (gr_text "GeneSynth Motherboard" (at 143.51 128.778) (layer F.SilkS)
+    (effects (font (size 1.2 1.2) (thickness 0.3)))
   )
   (gr_text GND (at 155.448 113.284 90) (layer F.SilkS)
@@
   (segment (start 126.033783 95.365) (end 134.912199 104.243416) (width 0.508) (layer F.Cu) (net 41))
   (segment (start 126.033783 94.107) (end 126.033783 95.365) (width 0.508) (layer F.Cu) (net 41))
+  (segment (start 141.224 120.904) (end 141.224 124.714) (width 0.508) (layer B.Cu) (net 41))
   (segment (start 149.9706 93.9636) (end 150.114 94.107) (width 0.508) (layer F.Cu) (net 42))
   (segment (start 149.9706 89.887) (end 149.9706 93.9636) (width 0.508) (layer F.Cu) (net 42))
-  (segment (start 146.6181 86.487) (end 149.9706 89.8395) (width 0.508) (layer F.Cu) (net 42))
-  (segment (start 149.9706 89.8395) (end 149.9706 89.887) (width 0.508) (layer F.Cu) (net 42))
-  (segment (start 140.4342 86.487) (end 146.6181 86.487) (width 0.508) (layer F.Cu) (net 42))
   (segment (start 151.372 94.107) (end 150.114 94.107) (width 0.508) (layer F.Cu) (net 42))
   (segment (start 157.357 100.092) (end 151.372 94.107) (width 0.508) (layer F.Cu) (net 42))
-  (segment (start 140.716 122.936) (end 138.684 120.904) (width 0.508) (layer B.Cu) (net 42))
   (segment (start 150.114 100.584) (end 146.558 104.14) (width 0.508) (layer B.Cu) (net 42))
   (segment (start 146.558 121.92) (end 145.542 122.936) (width 0.508) (layer B.Cu) (net 42))
   (segment (start 146.558 104.14) (end 146.558 121.92) (width 0.508) (layer B.Cu) (net 42))
-  (segment (start 145.542 122.936) (end 140.716 122.936) (width 0.508) (layer B.Cu) (net 42))
   (segment (start 157.357 100.584) (end 150.114 100.584) (width 0.508) (layer B.Cu) (net 42))
+  (segment (start 142.786199 125.945801) (end 143.218001 125.513999) (width 0.508) (layer B.Cu) (net 42))
+  (segment (start 140.632735 125.945801) (end 142.786199 125.945801) (width 0.508) (layer B.Cu) (net 42))
+  (segment (start 143.218001 125.513999) (end 144.018 124.714) (width 0.508) (layer B.Cu) (net 42))
+  (segment (start 138.684 123.997066) (end 140.632735 125.945801) (width 0.508) (layer B.Cu) (net 42))
+  (segment (start 138.684 120.904) (end 138.684 123.997066) (width 0.508) (layer B.Cu) (net 42))
+  (segment (start 145.542 123.19) (end 144.018 124.714) (width 0.508) (layer B.Cu) (net 42))
+  (segment (start 145.542 122.936) (end 145.542 123.19) (width 0.508) (layer B.Cu) (net 42))
+  (segment (start 143.548 87.884) (end 142.24 87.884) (width 0.508) (layer F.Cu) (net 42))
+  (segment (start 148.0151 87.884) (end 143.548 87.884) (width 0.508) (layer F.Cu) (net 42))
+  (segment (start 149.9706 89.8395) (end 148.0151 87.884) (width 0.508) (layer F.Cu) (net 42))
+  (segment (start 149.9706 89.887) (end 149.9706 89.8395) (width 0.508) (layer F.Cu) (net 42))
   (segment (start 149.86 111.76) (end 149.86 121.163092) (width 0.1778) (layer F.Cu) (net 43))
   (segment (start 149.86 121.163092) (end 149.854908 121.163092) (width 0.1778) (layer F.Cu) (net 43))
